File: V1.3/lightsounds.kicad_sch (KiCad schematic)
At the start: 30 parts, among them J1 Conn_01x03_Male, J2 Conn_01x03_Female, SW1 SW_DIP_x04, T1 AO3400A, T2 AO3400A, T5 AO3400A, T6 AO3400A

Commit message: fixing edges and connecting all pieces
Changed lines of the file:
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@@
+    (stroke (width 0) (type default) (color 0 0 0 0))
+  )
+  (wire (pts (xy 72.39 71.12) (xy 86.36 71.12))
     (stroke (width 0) (type default) (color 0 0 0 0))
   )
@@
   )
   (wire (pts (xy 52.07 62.23) (xy 52.07 63.5))
-    (stroke (width 0) (type default) (color 0 0 0 0))
-  )
-  (wire (pts (xy 72.39 71.12) (xy 74.93 71.12))
     (stroke (width 0) (type default) (color 0 0 0 0))
   )
@@
     (effects (font (size 2 2) (thickness 0.4) bold) (justify left bottom))
   )
+  (label "bypass" (at 71.12 71.12 270)
+    (effects (font (size 1.27 1.27)) (justify right bottom))
+  )
   (label "dcp1" (at 234.95 73.66 180)
     (effects (font (size 1.27 1.27)) (justify right bottom))
@@
     )
   )
-  (global_label "read-bypass" (shape input) (at 74.93 71.12 0) (fields_autoplaced)
+  (global_label "read-bypass" (shape input) (at 86.36 71.12 0) (fields_autoplaced)
     (effects (font (size 1.27 1.27)) (justify left))
-    (property "Intersheet References" "${INTERSHEET_REFS}" (id 0) (at 89.5593 71.0406 0)
+    (property "Intersheet References" "${INTERSHEET_REFS}" (id 0) (at 100.9893 71.0406 0)
       (effects (font (size 1.27 1.27)) (justify left) hide)
     )
