File: V1.3/mainslevelcontrol.kicad_sch (KiCad schematic)
At the start: 0 parts

Commit message: update v1.3 schematic documentation
Other:
- note added: "Mains Level Control"
- note added: "Stage 1"
- note added: "Stage 2"
- note added: "Stage 3"
- note added: "The original version of these tool controllers (before this design) required that this mains-level circuit be built by hand, every time. The goal here is to build a latching relay system from non-latching relays, with the added benefit of available E-Stops. Although a bit redundant, this design breaks up the control of power-access to a tool into three stages: --> 1) Small relays that are control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"
- note added: "This includes both logic- level relays circuits. The page also shows the 5VDC sealed transformer and a simple 'sanity check' power LED :)"
- note added: "This includes the one mains-controlled relay. Also, the logic of the main latching circuit is outlined on this page. The fuses are included here."
- note added: "With an off-board contactor this shows the logical loop that connects to the device. The screw-terminal connectors are also shown on this page."
Changed lines of the file:
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@@
     (company "Corey Rice & MakeHaven")
+  )
+  (text "With an off-board contactor\nthis shows the logical loop \nthat connects to the device.\n\nThe screw-terminal connectors\nare also shown on this page."
+    (at 196.85 163.83 0)
+    (effects (font (size 2.5 2.5)) (justify left bottom))
+  )
+  (text "This includes the one \nmains-controlled relay.\n\nAlso, the logic of the \nmain latching circuit is \noutlined on this page.\n\nThe fuses are included here."
+    (at 110.49 170.18 0)
+    (effects (font (size 2.5 2.5)) (justify left bottom))
+  )
+  (text "Stage 3" (at 210.82 116.84 0)
+    (effects (font (size 3.5 3.5) (thickness 0.7) bold) (justify left bottom))
+  )
+  (text "Mains Level Control" (at 48.26 49.53 0)
+    (effects (font (size 12 12) (thickness 2.4) bold italic) (justify left bottom))
+  )
+  (text "Stage 2" (at 120.65 118.11 0)
+    (effects (font (size 3.5 3.5) (thickness 0.7) bold) (justify left bottom))
+  )
+  (text "The original version of these tool controllers (before this design) \nrequired that this mains-level circuit be built by hand, every time. \n\nThe goal here is to build a latching relay system from non-latching relays, with the added benefit of available E-Stops. \nAlthough a bit redundant, this design breaks up the control of power-access to a tool into three stages: \n\n--> 1) Small relays that are controlled by a microcontroller, which allow access to use tool\n\n--> 2) A larger relay that is triggered and controls mains-level voltage (also has 110 & 220 versions)\n\n--> 3) An off-board contactor that actually transmits the full power needs of the tool"
+    (at 24.13 100.33 0)
+    (effects (font (size 2.5 2.5)) (justify left bottom))
+  )
+  (text "This includes both logic-\nlevel relays circuits.\n\nThe page also shows the \n5VDC sealed transformer \nand a simple 'sanity \ncheck' power LED :)"
+    (at 22.86 167.64 0)
+    (effects (font (size 2.5 2.5)) (justify left bottom))
+  )
+  (text "Stage 1" (at 31.75 116.84 0)
+    (effects (font (size 3.5 3.5) (thickness 0.7) bold) (justify left bottom))
   )
   (sheet (at 213.36 120.65) (size 17.78 13.97) (fields_autoplaced)
