File: V1.3/mh-custom-v1.3.kicad_sch (KiCad schematic)
At the start: 0 parts

Commit message: update v1.3 schematic documentation
Other:
- note added: "This device is intended to help simplify the process of setting up and managing tool authorization control, in a shared workshop environment. Specifically, this is designed for use at MakeHaven, in New Haven, Connecticut, USA from a previous solution. The circuit board shown here includes a place for an ESP32-DEVKITC-V4+ microcontroller (with wifi) to sit into place, and manage the functions of t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"
- note added: "This section covers everything that happens at the AC power level: anywhere from 100VAC to 240VAC, provided the correct configuration. There is only a single relay changed to cover voltage this range. All the panel-mount buttons, relays and Emergency Stops that ensure primary function of the tool-control are included here."
- note added: "This section of the schematic covers everything that happens at 3.3VDC or 5VDC, including the microcontroller, peripherals, and some of the simple circuits needed to support the operation Power for this section is provided by a sealed switching transformer soldered onto the board."
- note added: "ToolAuth Hardware | Overview"
- note removed: "OpenShop Hardware | Overview"
- note removed: "This 'OpenShop' device is intended to help simplify the process of setting up and managing tool authorization control, in a shared workshop environment. Specifically, this is designed for use at MakeHaven, in New Haven, Connecticut, USA from a previous solution. The circuit board shown here includes a place for an ESP32-DEVKITC-V4+ microcontroller (with wifi) to sit into place, and manage the fun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"
- note removed: "This section of the schematic covers everything that happens at 3.3VDC or 5VDC, including the microcontroller, peripherals, and some of the simple circuits needed to support the operation of the device while in full operation. Power for this section of the circuit is provided by a sealed switching transformer soldered onto the board. The one other crossover circuit is the bypass switch, which ope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"
- note removed: "This section of the schematic covers everything that happens at the AC power level, and this can be at anywhere from 100VAC to 240VAC, provided the correct configuration. There is only a single relay that needs changed to cover this range, and all the other components in this section are tolerant of this span of voltages. The things included here are all the panel-mount buttons, relays and Emerge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"
Changed lines of the file:
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@@
     (comment 1 "Highest Level Overview")
   )
-  (wire (pts (xy 91.44 139.7) (xy 193.04 139.7))
+  (wire (pts (xy 91.44 149.86) (xy 193.04 149.86))
     (stroke (width 0) (type default) (color 0 0 0 0))
   )
-  (wire (pts (xy 91.44 130.81) (xy 193.04 130.81))
+  (wire (pts (xy 91.44 140.97) (xy 193.04 140.97))
     (stroke (width 0) (type default) (color 0 0 0 0))
   )
-  (text "OpenShop Hardware | Overview" (at 40.64 39.37 0)
-    (effects (font (size 5 5) (thickness 0.5) bold) (justify left bottom))
+  (text "ToolAuth Hardware | Overview" (at 22.86 36.83 0)
+    (effects (font (size 10 10) (thickness 2) bold italic) (justify left bottom))
   )
   (text "Mains Level Control" (at 184.15 93.98 0)
@@
     (effects (font (size 3.5 3.5) bold) (justify left bottom))
   )
-  (text "This section of the schematic covers everything that happens at \n3.3VDC or 5VDC, including the microcontroller, peripherals, and \nsome of the simple circuits needed to support the operation of \nthe device while in full operation. Power for this section of \nthe circuit is provided by a sealed switching transformer soldered \nonto the board. The one other crossover circuit  is the bypass \nswitch, which operates on a 5VDC circuit, but activates a relay \nthat enables the entirety of the mains level control. \n"
-    (at 34.29 120.65 0)
-    (effects (font (size 1.75 1.75)) (justify left bottom))
+  (text "This section of the schematic covers everything \nthat happens at 3.3VDC or 5VDC, including the \nmicrocontroller, peripherals, and some of the \nsimple circuits needed to support the operation \n\nPower for this section is provided by a sealed \nswitching transformer soldered onto the board. "
+    (at 29.21 128.27 0)
+    (effects (font (size 2.5 2.5)) (justify left bottom))
   )
-  (text "This 'OpenShop' device is intended to help simplify the process of setting up and managing tool authorization control, in a shared workshop environment. \nSpecifically, this is designed for use at MakeHaven, in New Haven, Connecticut, USA from a previous solution. The circuit board shown here includes a \nplace for an ESP32-DEVKITC-V4+ microcontroller (with wifi) to sit into place, and manage the functions of theboard and ultimately control access to \npower a tool. However, through experience, MakeHaven knows it is also important to have a completely analog work-around to enable tools when the network-\nbased system goes down. For that reason, the tool can be granted unfiltered access with a bypass key, and this works regardless of the microcontroller, \neven if the microcontroller is completely absent. \n\nThis schematic is broken into several pages to better clarify the circuit surrounding each of the components. Global Labels have been heavily used to \nshow connections that span across sections and pages. Some of the components are shown for reference to be used with the circuit board, but are not \nthemselves on the circuit board design. \n"
-    (at 35.56 72.39 0)
-    (effects (font (size 1.75 1.75)) (justify left bottom))
+  (text "This device is intended to help simplify the process of setting up and managing tool authorization \ncontrol, in a shared workshop environment. \n\nSpecifically, this is designed for use at MakeHaven, in New Haven, Connecticut, USA from a previous\nsolution. The circuit board shown here includes a place for an ESP32-DEVKITC-V4+ microcontroller \n(with wifi) to sit into place, and manage the functions of theboard and ultimately control access \nto power a tool. This schematic is broken into several pages to better clarify the circuit.\n"
+    (at 41.91 71.12 0)
+    (effects (font (size 2.5 2.5)) (justify left bottom))
   )
-  (text "This section of the schematic covers everything that happens at \nthe AC power level, and this can be at anywhere from 100VAC to \n240VAC, provided the correct configuration. There is only a single \nrelay that needs changed to cover this range, and all the other \ncomponents in this section are tolerant of this span of voltages. \nThe things included here are all the panel-mount buttons, relays \nand Emergency Stops that ensure the ToolAuth system can function \nsafely in a workshop.\n"
-    (at 165.1 120.65 0)
-    (effects (font (size 1.75 1.75)) (justify left bottom))
+  (text "This section covers everything that happens at \nthe AC power level: anywhere from 100VAC to \n240VAC, provided the correct configuration. \n\nThere is only a single relay changed to cover \nvoltage this range. All the panel-mount buttons, \nrelays and Emergency Stops that ensure primary\nfunction of the tool-control are included here."
+    (at 161.29 130.81 0)
+    (effects (font (size 2.5 2.5)) (justify left bottom))
   )
-  (text "Based Around ESP32-DEVKITC-V4+ board" (at 26.67 161.29 0)
+  (text "Based Around ESP32-DEVKITC-V4+ board" (at 27.94 191.77 0)
     (effects (font (size 3 3) (thickness 0.6) bold italic) (justify left bottom))
   )
-  (hierarchical_label "5VDC Power" (shape output) (at 193.04 130.81 0)
+  (hierarchical_label "5VDC Power" (shape output) (at 193.04 140.97 0)
     (effects (font (size 1.75 1.75)) (justify left))
   )
-  (hierarchical_label "Bypass Control" (shape output) (at 91.44 139.7 180)
+  (hierarchical_label "Bypass Control" (shape output) (at 91.44 149.86 180)
     (effects (font (size 1.75 1.75)) (justify right))
   )
-  (hierarchical_label "Bypass Control" (shape input) (at 193.04 139.7 0)
+  (hierarchical_label "Bypass Control" (shape input) (at 193.04 149.86 0)
     (effects (font (size 1.75 1.75)) (justify left))
   )
-  (hierarchical_label "5VDC Power" (shape input) (at 91.44 130.81 180)
+  (hierarchical_label "5VDC Power" (shape input) (at 91.44 140.97 180)
     (effects (font (size 1.75 1.75)) (justify right))
   )
-  (sheet (at 49.53 127) (size 41.91 24.13) (fields_autoplaced)
+  (sheet (at 49.53 137.16) (size 41.91 24.13) (fields_autoplaced)
     (stroke (width 0.1524) (type solid) (color 0 0 0 0))
     (fill (color 0 0 0 0.0000))
-    (property "Sheet name" "microcontroller" (id 0) (at 49.53 126.2884 0)
+    (property "Sheet name" "microcontroller" (id 0) (at 49.53 136.4484 0)
       (effects (font (size 1.27 1.27)) (justify left bottom))
     )
-    (property "Sheet file" "microcontroller.kicad_sch" (id 1) (at 49.53 151.7146 0)
+    (property "Sheet file" "microcontroller.kicad_sch" (id 1) (at 49.53 161.8746 0)
       (effects (font (size 1.27 1.27)) (justify left top))
     )
   )
-  (sheet (at 193.04 127) (size 38.1 24.13) (fields_autoplaced)
+  (sheet (at 193.04 137.16) (size 38.1 24.13) (fields_autoplaced)
     (stroke (width 0.1524) (type solid) (color 0 0 0 0))
     (fill (color 0 0 0 0.0000))
-    (property "Sheet name" "mainslevelcontrol" (id 0) (at 193.04 126.2884 0)
+    (property "Sheet name" "mainslevelcontrol" (id 0) (at 193.04 136.4484 0)
       (effects (font (size 1.27 1.27)) (justify left bottom))
     )
-    (property "Sheet file" "mainslevelcontrol.kicad_sch" (id 1) (at 193.04 151.7146 0)
+    (property "Sheet file" "mainslevelcontrol.kicad_sch" (id 1) (at 193.04 161.8746 0)
       (effects (font (size 1.27 1.27)) (justify left top))
     )
