File: V1.3/microcontroller.kicad_sch (KiCad schematic)
At the start: 0 parts

Commit message: update v1.3 schematic documentation
Other:
- note added: "Lights, Sounds & Status"
- note removed: "Lights, Sounds & Buttons"
Changed lines of the file:
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@@
     (company "Corey Rice & MakeHaven")
   )
-  (text "This shows the relationships between all components running at 3.3VDC or 5VDC on the board. These are all on the 'low voltage' \nside of the board. These are all united in their service to the ESP32-DEVKITC-V4+ board, but that board itself is removable \n(for ease of programming and switching out the controller, without needing to rewire the tools). "
-    (at 35.56 40.64 0)
-    (effects (font (size 1.75 1.75)) (justify left bottom))
+  (text "This shows the relationships between all components running at 3.3VDC or 5VDC on the board. \nThese are all on the 'low voltage' side of the board. These are all united in their service \nto the ESP32-DEVKITC-V4+ board, but that board itself is removable (for ease of programming \nand switching out the controller, without needing to rewire the tools). "
+    (at 33.02 49.53 0)
+    (effects (font (size 2.5 2.5)) (justify left bottom))
   )
   (text "This is a collection of the simple circuits \nthat translate between voltage levels, break \nout the programming buttons for the ESP32, \ndescribe the DIP switches for configuration \nself-description, control the buzzer, and \ncontrol the indicator LEDs. Many of these \ncircuits use the 3.3V from the ESP32's \nonboard regulator.\n"
@@
     (effects (font (size 1.75 1.75)) (justify left bottom))
   )
-  (text "Lights, Sounds & Buttons" (at 142.24 127 0)
+  (text "Lights, Sounds & Status" (at 142.24 127 0)
     (effects (font (size 3.5 3.5) bold) (justify left bottom))
   )
